Commit message: 添加转换

File: install/lidar/share/lidar/urdf/robot.urdf.xacro (robot description, xacro)
@@ -1,4 +1,4 @@
 <?xml version="1.0"?>
-<robot name="robot">
+<robot xmlns:xacro="http://www.ros.org/wiki/xacro" name="robot">
   <!-- Robot Footprint -->
   <link name="base_footprint"/>
@@ -143,4 +143,5 @@
       <axis xyz="0 1 0" />
       <limit effort="20" velocity="10"/>  <!-- 添加努力限制，支持扭矩 -->
+      <dynamics damping="0.0" friction="0.0"/>
   </joint>
   <joint name="right_wheel_joint" type="continuous">
@@ -150,4 +151,5 @@
       <axis xyz="0 1 0" />
       <limit effort="20" velocity="10"/>  <!-- 添加努力限制，支持扭矩 -->
+      <dynamics damping="0.0" friction="0.0"/>
   </joint>
   <link name="caster_link">
@@ -200,5 +202,5 @@
       <update_rate>100</update_rate>
       <visualize>true</visualize>
-      <topic>/modle/robot/imu</topic>  <!-- 输出话题 -->
+      <topic>/robot/imu</topic>  <!-- 输出话题 -->
       <imu>
         <angular_velocity>
@@ -263,5 +265,5 @@
       <visualize>true</visualize>
       <update_rate>5</update_rate>
-      <topic>/model/robot/scan</topic>  <!-- 输出话题 -->
+      <topic>/scan</topic>  <!-- 输出话题 -->
       <lidar>  <!-- 替换原 <ray> -->
         <scan>
@@ -296,10 +298,12 @@
       <remapping>odom:=odom</remapping>
     </ros>
+    <publish_joint_state>true</publish_joint_state>
+    <joint_state_topic>/joint_states</joint_state_topic>
     <!-- 左右轮关节名（必须和你 URDF 里完全一模一样！） -->
     <left_joint>left_wheel_joint</left_joint>
     <right_joint>right_wheel_joint</right_joint>
     <!-- 物理参数（必须和实际模型一致！） -->
-    <wheel_separation>0.38</wheel_separation>      <!-- 两轮中心距离，单位：米 -->
-    <wheel_diameter>0.065</wheel_diameter>         <!-- 轮子直径，单位：米 -->
+    <wheel_separation>0.20</wheel_separation>      <!-- 两轮中心距离，单位：米 -->
+    <wheel_diameter>0.064</wheel_diameter>         <!-- 轮子直径，单位：米 -->
     <!-- 限制（根据你的电机调整） -->
     <max_wheel_torque>20</max_wheel_torque>
@@ -309,6 +313,6 @@
     <publish_odom>true</publish_odom>
     <publish_odom_tf>true</publish_odom_tf>        <!-- 发布 odom → base_footprint 的 TF -->
-    <publish_wheel_tf>false</publish_wheel_tf>     <!-- 一般设 false，轮子 TF 不需要 -->
-    <!-- TF 帧名（必须和你 URDF + base_footprint 一致！） -->
+    <publish_wheel_tf>true</publish_wheel_tf>     <!-- 一般设 false，轮子 TF 不需要 -->
+    <!-- TF 帧名 -->
     <odometry_frame>odom</odometry_frame>
     <robot_base_frame>base_footprint</robot_base_frame>
@@ -316,11 +320,12 @@
     <odom_publisher_frequency>50</odom_publisher_frequency>
   </plugin>
-  <!-- 2. 关节状态发布插件（可选，如果你桥接了 /joint_states 就留着） -->
-  <plugin filename="gz-sim-joint-state-publisher-system" name="gz::sim::systems::JointStatePublisher">
+  <!-- 2. 关节状态发布插件 -->
+  <!-- <plugin filename="gz-sim-joint-state-publisher-system"
+          name="gz::sim::systems::JointStatePublisher">
     <topic>/joint_states</topic>
     <joint_name>left_wheel_joint</joint_name>
     <joint_name>right_wheel_joint</joint_name>
-    <!-- 如果你还有云台等关节，继续加 <joint_name>xxx</joint_name> -->
-  </plugin>
+    <include_all_joints>true</include_all_joints>
+  </plugin> -->
 </gazebo>
 </robot>

File: src/lidar/urdf/robot.urdf.xacro (robot description, xacro)
@@ -1,11 +1,6 @@
 <?xml version="1.0"?>
-<robot name="robot">
+<robot xmlns:xacro="http://www.ros.org/wiki/xacro" name="robot">
   <!-- Robot Footprint -->
   <link name="base_footprint"/>
-  <joint name="base_joint" type="fixed">
-    <parent link="base_footprint"/>
-    <child link="base_link"/>
-    <origin xyz="0.0 0.0 0.076" rpy="0 0 0"/>
-  </joint>
   <!-- base link -->
   <link name="base_link">
@@ -58,10 +53,4 @@
     </inertial>
   </link>
-  <!-- laser joint -->
-  <joint name="laser_joint" type="fixed">
-      <parent link="base_link" />
-      <child link="laser_link" />
-      <origin xyz="0 0 0.075" />
-  </joint>
   <link name="imu_link">
     <visual>
@@ -82,10 +71,4 @@
     </inertial>
   </link>
-  <!-- imu joint -->
-  <joint name="imu_joint" type="fixed">
-      <parent link="base_link" />
-      <child link="imu_link" />
-      <origin xyz="0 0 0.02" />
-  </joint>
   <link name="left_wheel_link">
       <visual>
@@ -136,4 +119,22 @@
       </inertial>
   </link>
+  <!-- base_joint -->
+  <joint name="base_joint" type="fixed">
+    <parent link="base_footprint"/>
+    <child link="base_link"/>
+    <origin xyz="0.0 0.0 0.076" rpy="0 0 0"/>
+  </joint>
+  <!-- laser joint -->
+  <joint name="laser_joint" type="fixed">
+      <parent link="base_link" />
+      <child link="laser_link" />
+      <origin xyz="0 0 0.075" />
+  </joint>
+  <!-- imu joint -->
+  <joint name="imu_joint" type="fixed">
+      <parent link="base_link" />
+      <child link="imu_link" />
+      <origin xyz="0 0 0.02" />
+  </joint>
   <joint name="left_wheel_joint" type="continuous">
       <parent link="base_link" />
@@ -142,4 +143,5 @@
       <axis xyz="0 1 0" />
       <limit effort="20" velocity="10"/>  <!-- 添加努力限制，支持扭矩 -->
+      <dynamics damping="0.0" friction="0.0"/>
   </joint>
   <joint name="right_wheel_joint" type="continuous">
@@ -149,4 +151,5 @@
       <axis xyz="0 1 0" />
       <limit effort="20" velocity="10"/>  <!-- 添加努力限制，支持扭矩 -->
+      <dynamics damping="0.0" friction="0.0"/>
   </joint>
   <link name="caster_link">
@@ -199,5 +202,5 @@
       <update_rate>100</update_rate>
       <visualize>true</visualize>
-      <topic>/modle/robot/imu</topic>  <!-- 输出话题 -->
+      <topic>/robot/imu</topic>  <!-- 输出话题 -->
       <imu>
         <angular_velocity>
@@ -262,5 +265,5 @@
       <visualize>true</visualize>
       <update_rate>5</update_rate>
-      <topic>/model/robot/scan</topic>  <!-- 输出话题 -->
+      <topic>/scan</topic>  <!-- 输出话题 -->
       <lidar>  <!-- 替换原 <ray> -->
         <scan>
@@ -286,28 +289,43 @@
   </gazebo>
   <!-- 模型级插件：差速驱动和关节状态发布 -->
-  <gazebo>
-    <!-- 差速驱动插件 -->
-    <plugin filename="gz-sim-diff-drive-system" name="gz::sim::systems::DiffDrive">
-      <left_joint>left_wheel_joint</left_joint>
-      <right_joint>right_wheel_joint</right_joint>
-      <wheel_separation>0.2</wheel_separation>
-      <wheel_diameter>0.065</wheel_diameter>
-      <max_wheel_torque>20</max_wheel_torque>
-      <max_linear_acceleration>1.0</max_linear_acceleration>
-      <topic>cmd_vel</topic>
-      <odom_topic>odom</odom_topic>
-      <frame_id>odom</frame_id>
-      <child_frame_id>base_footprint</child_frame_id>
-      <odom_publisher_frequency>30</odom_publisher_frequency>
-      <publish_odom>true</publish_odom>
-      <publish_odom_tf>true</publish_odom_tf>
-      <publish_wheel_tf>false</publish_wheel_tf>
-    </plugin>
-    <!-- 关节状态发布插件 -->
-    <plugin filename="gz-sim-joint-state-publisher-system" name="gz::sim::systems::JointStatePublisher">
-      <topic>joint_states</topic>
-      <joint_name>left_wheel_joint</joint_name>
-      <joint_name>right_wheel_joint</joint_name>
-    </plugin>
-  </gazebo>
+<gazebo>
+  <!-- 1. 差速驱动插件（官方最新版） -->
+  <plugin filename="gz-sim-diff-drive-system" name="gz::sim::systems::DiffDrive">
+    <!-- ROS 2 桥接（可选，如果你用了 ros_gz_bridge） -->
+    <ros>
+      <namespace>/</namespace>          <!-- 建议改成 /robot1 之类避免多机器人冲突 -->
+      <remapping>cmd_vel:=cmd_vel</remapping>
+      <remapping>odom:=odom</remapping>
+    </ros>
+    <publish_joint_state>true</publish_joint_state>
+    <joint_state_topic>/joint_states</joint_state_topic>
+    <!-- 左右轮关节名（必须和你 URDF 里完全一模一样！） -->
+    <left_joint>left_wheel_joint</left_joint>
+    <right_joint>right_wheel_joint</right_joint>
+    <!-- 物理参数（必须和实际模型一致！） -->
+    <wheel_separation>0.20</wheel_separation>      <!-- 两轮中心距离，单位：米 -->
+    <wheel_diameter>0.064</wheel_diameter>         <!-- 轮子直径，单位：米 -->
+    <!-- 限制（根据你的电机调整） -->
+    <max_wheel_torque>20</max_wheel_torque>
+    <max_wheel_acceleration>5.0</max_wheel_acceleration>
+    <max_linear_acceleration>2.0</max_linear_acceleration>
+    <!-- 发布设置（关键！） -->
+    <publish_odom>true</publish_odom>
+    <publish_odom_tf>true</publish_odom_tf>        <!-- 发布 odom → base_footprint 的 TF -->
+    <publish_wheel_tf>true</publish_wheel_tf>     <!-- 一般设 false，轮子 TF 不需要 -->
+    <!-- TF 帧名 -->
+    <odometry_frame>odom</odometry_frame>
+    <robot_base_frame>base_footprint</robot_base_frame>
+    <!-- 发布频率 -->
+    <odom_publisher_frequency>50</odom_publisher_frequency>
+  </plugin>
+  <!-- 2. 关节状态发布插件 -->
+  <!-- <plugin filename="gz-sim-joint-state-publisher-system"
+          name="gz::sim::systems::JointStatePublisher">
+    <topic>/joint_states</topic>
+    <joint_name>left_wheel_joint</joint_name>
+    <joint_name>right_wheel_joint</joint_name>
+    <include_all_joints>true</include_all_joints>
+  </plugin> -->
+</gazebo>
 </robot>
